File: Hardware/IceBoard-Rev3.sch (EAGLE design)
At the start: 12 parts

Commit message: IceBoard Rev3 Hardware
Parts:
- added R1, R2: 10k, resistor:R-US_R0805
- added TEMP2, TEMP3: 22-23-2021, con-molex:22-23-2021
Connections:
- new net N$10: CH5-2.S, U$1.D12
- new net N$12: CH4-2.S, U$1.D8
- new net N$13: CH3-2.S, U$1.D7
- new net N$14: CH2-2-2.S, U$1.D4
- new net N$15: CH1-2.S, U$1.D2
- new net N$16: U$1.A2
- new net N$18: R2.1, TEMP3-1.S, U$1.A5
- new net N$7: R3.1, TEMP2-1.S, U$1.A6
- new net N$9: CH6-2.S, U$1.D13
- net 10K: now also TEMP1-2.S, TEMP2-2.S, TEMP3-2.S; no longer R3.1, TEMP1-1.S
- net GND: now also R1.2, R2.2, R3.2; no longer TEMP1-2.S
- net N$11: now also R1.1, TEMP1-1.S; no longer R3.2
Other:
- moved on the sheet: R3

Commit message: IceBoard Rev3 Hardware
Changed lines of the file:
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@@
 <grid distance="0.1" unitdist="inch" unit="inch" style="lines" multiple="1" display="no" altdistance="0.01" altunitdist="inch" altunit="inch"/>
 <layers>
-<layer number="1" name="Top" color="4" fill="10" visible="no" active="no"/>
+<layer number="1" name="Top" color="4" fill="1" visible="no" active="no"/>
 <layer number="16" name="Bottom" color="1" fill="1" visible="no" active="no"/>
 <layer number="17" name="Pads" color="2" fill="1" visible="no" active="no"/>
@@
 <layer number="48" name="Document" color="7" fill="1" visible="no" active="no"/>
 <layer number="49" name="Reference" color="7" fill="1" visible="no" active="no"/>
-<layer number="51" name="tDocu" color="26" fill="1" visible="no" active="no"/>
+<layer number="51" name="tDocu" color="7" fill="1" visible="no" active="no"/>
 <layer number="52" name="bDocu" color="7" fill="1" visible="no" active="no"/>
 <layer number="90" name="Modules" color="5" fill="1" visible="yes" active="yes"/>
@@
 <junction x="-12.7" y="111.76"/>
 <junction x="-7.62" y="111.76"/>
-</segment>
-</net>
+<junction x="20.32" y="111.76"/>
+<junction x="88.9" y="111.76"/>
+<junction x="20.32" y="129.54"/>
+</segment>
+</net>

Commit message: rev3 board
Parts:
- added H1, H2, H3, H4: MOUNT-PAD-ROUND3.3, holes:MOUNT-PAD-ROUND3.3
Changed lines of the file:
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@@
 <part name="TEMP2" library="con-molex" deviceset="22-23-2021" device=""/>
 <part name="TEMP3" library="con-molex" deviceset="22-23-2021" device=""/>
+<part name="H1" library="holes" deviceset="MOUNT-PAD-ROUND" device="3.3"/>
+<part name="H2" library="holes" deviceset="MOUNT-PAD-ROUND" device="3.3"/>
+<part name="H3" library="holes" deviceset="MOUNT-PAD-ROUND" device="3.3"/>
+<part name="H4" library="holes" deviceset="MOUNT-PAD-ROUND" device="3.3"/>
 </parts>
 <sheets>
@@
 <instance part="TEMP3" gate="-1" x="12.7" y="0"/>
 <instance part="TEMP3" gate="-2" x="15.24" y="-5.08"/>
+<instance part="H1" gate="G$1" x="-35.56" y="142.24"/>
+<instance part="H2" gate="G$1" x="-35.56" y="134.62"/>
+<instance part="H3" gate="G$1" x="-35.56" y="127"/>
+<instance part="H4" gate="G$1" x="-35.56" y="119.38"/>
 </instances>
 <busses>
@@
 <junction x="20.32" y="129.54"/>
 </segment>
+<segment>
+<wire x1="-35.56" y1="127" x2="-48.26" y2="127" width="0.1524" layer="91"/>
+</segment>
+<segment>
+<wire x1="-35.56" y1="142.24" x2="-48.26" y2="142.24" width="0.1524" layer="91"/>
+</segment>
+<segment>
+<wire x1="-35.56" y1="134.62" x2="-48.26" y2="134.62" width="0.1524" layer="91"/>
+</segment>
+<segment>
+<wire x1="-35.56" y1="119.38" x2="-48.26" y2="119.38" width="0.1524" layer="91"/>
+</segment>
 </net>
